File: CAD/tmc_2300_standalone_bob/tmc_2300_standalone_bob.kicad_pcb (KiCad board)
At the start: 4 copper layers, 28.8 x 25.4 mm, 35 parts, among them IC1 TMC2300, J1 Conn_01x04_Pin, J2 Conn_01x08_Pin, J3 Conn_01x08_Pin, J4 53261-0471

Commit message: fixed schematic
Parts:
- D1: value 0603/LED -> LED; footprint Resistor_SMD:R_0603_1608Metric -> LED_SMD:LED_0603_1608Metric
- D2: value white/0603 -> LED
- moved TP5 0.96 mm to (159.6, 84.0)
- renumbered DIAG to TP1, OA1 to TP4, OA2 to TP5, OB1 to TP6, OB2 to TP7
Routing:
- net /OA2: track 20.0 -> 20.9 mm
- net +3.3V: track 8.03 -> 8.56 mm
- net GND: track 1.16 -> 0.88 mm, vias 30 -> 31
