File: CAD/tmc_2300_standalone_bob/tmc_2300_standalone_bob.kicad_sch (KiCad schematic)
At the start: 33 parts, among them IC1 TMC2300, J1 Conn_01x04_Pin, J2 Conn_01x08_Pin, J3 Conn_01x08_Pin, J4 53261-0471

Commit message: fixed schematic
Parts:
- D1: value 0603/LED -> LED; footprint Resistor_SMD:R_0603_1608Metric -> LED_SMD:LED_0603_1608Metric; Info Green -> (none); color (none) -> green
- D2: value white/0603 -> LED; color (none) -> red
Changed lines of the file:
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@@
+    )
+  )
+  (symbol (lib_id "Device:LED") (at 45.72 95.25 90) (unit 1)
+    (in_bom yes) (on_board yes) (dnp no)
+    (property "Reference" "D1" (at 49.53 95.5675 90)
+      (effects (font (size 1.27 1.27)) (justify right))
+    )
+    (property "Value" "LED" (at 49.53 98.1075 90)
+      (effects (font (size 1.27 1.27)) (justify right))
+    )
+    (property "Footprint" "LED_SMD:LED_0603_1608Metric" (at 45.72 95.25 0)
+      (effects (font (size 1.27 1.27)) hide)
+    )
+    (property "Datasheet" "~" (at 45.72 95.25 0)
+      (effects (font (size 1.27 1.27)) hide)
+    )
+    (property "color" "green" (at 52.07 100.33 90)
+      (effects (font (size 1.27 1.27)))
+    )
+    (pin "1")
+    (pin "2")
+    (instances
+      (project "tmc_2300_standalone_bob"
+        (path "/52d152b1-d4bc-430c-a4a2-89987d55cda0"
+          (reference "D1") (unit 1)
+        )
+      )
     )
   )
@@
   )
   (symbol (lib_id "Connector:TestPoint") (at 171.45 76.2 0) (unit 1)
-    (in_bom yes) (on_board yes) (dnp no) (fields_autoplaced)
+    (in_bom yes) (on_board yes) (dnp no)
     (property "Reference" "TP1" (at 173.99 71.628 0)
-      (effects (font (size 1.27 1.27)) (justify left))
+      (effects (font (size 1.27 1.27)) (justify left) hide)
     )
     (property "Value" "TestPoint" (at 173.99 74.168 0)
@@
       (effects (font (size 1.27 1.27)) hide)
     )
-    (property "Feld4" "DIAG" (at 171.45 76.2 0)
-      (effects (font (size 1.27 1.27)) hide)
+    (property "Feld4" "DIAG" (at 171.45 71.12 0)
+      (effects (font (size 1.27 1.27)))
     )
     (pin "1")
@@
     )
   )
-  (symbol (lib_id "Device:LED") (at 171.45 82.55 90) (unit 1)
-    (in_bom yes) (on_board yes) (dnp no)
-    (property "Reference" "D2" (at 167.64 82.55 0)
-      (effects (font (size 0.9906 0.9906)))
-    )
-    (property "Value" "white/0603" (at 175.26 82.55 0)
-      (effects (font (size 0.9906 0.9906)))
-    )
-    (property "Footprint" "LED_SMD:LED_0603_1608Metric" (at 171.45 82.55 0)
-      (effects (font (size 1.27 1.27)) hide)
-    )
-    (property "Datasheet" "~" (at 171.45 82.55 0)
-      (effects (font (size 1.27 1.27)) hide)
-    )
-    (pin "1")
-    (pin "2")
-    (instances
-      (project "TMC2300-BOB v1.0"
-        (path "/25e9b056-4d94-493f-9a12-a9983474c725"
-          (reference "D2") (unit 1)
-        )
-      )
-      (project "tmc_2300_standalone_bob"
-        (path "/52d152b1-d4bc-430c-a4a2-89987d55cda0"
-          (reference "D2") (unit 1)
-        )
-      )
-    )
-  )
   (symbol (lib_id "power:GND") (at 240.03 53.34 0) (unit 1)
     (in_bom yes) (on_board yes) (dnp no)
@@
     )
   )
+  (symbol (lib_id "Device:LED") (at 171.45 82.55 90) (unit 1)
+    (in_bom yes) (on_board yes) (dnp no)
+    (property "Reference" "D2" (at 175.26 82.8675 90)
+      (effects (font (size 1.27 1.27)) (justify right))
+    )
+    (property "Value" "LED" (at 175.26 85.09 90)
+      (effects (font (size 1.27 1.27)) (justify right))
+    )
+    (property "Footprint" "LED_SMD:LED_0603_1608Metric" (at 171.45 82.55 0)
+      (effects (font (size 1.27 1.27)) hide)
+    )
+    (property "Datasheet" "~" (at 171.45 82.55 0)
+      (effects (font (size 1.27 1.27)) hide)
+    )
+    (property "color" "red" (at 176.53 87.63 90)
+      (effects (font (size 1.27 1.27)))
+    )
+    (pin "1")
+    (pin "2")
+    (instances
+      (project "tmc_2300_standalone_bob"
+        (path "/52d152b1-d4bc-430c-a4a2-89987d55cda0"
+          (reference "D2") (unit 1)
+        )
+      )
+    )
+  )
   (symbol (lib_id "Connector:TestPoint") (at 245.11 44.45 0) (unit 1)
-    (in_bom yes) (on_board yes) (dnp no) (fields_autoplaced)
+    (in_bom yes) (on_board yes) (dnp no)
     (property "Reference" "TP4" (at 247.65 39.878 0)
-      (effects (font (size 1.27 1.27)) (justify left))
+      (effects (font (size 1.27 1.27)) (justify left) hide)
     )
     (property "Value" "TestPoint" (at 247.65 42.418 0)
@@
       (effects (font (size 1.27 1.27)) hide)
     )
-    (property "Feld4" "OA1" (at 245.11 44.45 0)
-      (effects (font (size 1.27 1.27)) hide)
+    (property "Feld4" "OA1" (at 245.11 38.1 0)
+      (effects (font (size 1.27 1.27)))
     )
     (pin "1")
@@
         )
       )
-    )
-  )
-  (symbol (lib_id "Device:LED") (at 45.72 95.25 270) (mirror x) (unit 1)
-    (in_bom yes) (on_board yes) (dnp no)
-    (property "Reference" "D1" (at 41.91 95.25 0)
-      (effects (font (size 0.9906 0.9906)))
-    )
-    (property "Value" "0603/LED" (at 48.26 95.25 0)
-      (effects (font (size 0.9906 0.9906)))
-    )
-    (property "Footprint" "Resistor_SMD:R_0603_1608Metric" (at 45.72 95.25 0)
-      (effects (font (size 0.9906 0.9906)) hide)
-    )
-    (property "Datasheet" "~" (at 45.72 95.25 0)
-      (effects (font (size 0.9906 0.9906)) hide)
-    )
-    (property "Info" "Green" (at 49.53 95.25 0)
-      (effects (font (size 0.7874 0.7874)))
-    )
-    (pin "1")
-    (pin "2")
-    (instances
-      (project "TMC2300-BOB v1.0"
-        (path "/25e9b056-4d94-493f-9a12-a9983474c725"
-          (reference "D1") (unit 1)
-        )
-      )
-      (project "tmc_2300_standalone_bob"
-        (path "/52d152b1-d4bc-430c-a4a2-89987d55cda0"
-          (reference "D1") (unit 1)
-        )
-      )
-      (project "TMC2300-THERMO-BOB v2.0"
-        (path "/de4ac01b-f0de-4a2e-bc09-e05893b35240/00000000-0000-0000-0000-00005c8b1cdc"
-          (reference "D1") (unit 1)
-        )
-      )

Commit message: changed wrong resistor values in schematic
Parts:
- R1, R4: value 100k -> 1k
- R10: value 220 -> 1k
- R11, R12: value 220 -> 0.22
Changed lines of the file:
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@@
     (stroke (width 0) (type default))
+  )
+  (text_box "CHANGELOG \n\nREF 2:\n* Change R1 to use a 1k Resistor \n* Change R4, R10 to 1k\n* change R11, 12 to 0.22 Ohm "
+    (at -69.85 99.06 0) (size 69.85 40.64)
+    (stroke (width 0) (type default))
+    (fill (type none))
+    (effects (font (size 1.27 1.27)) (justify left top))
   )
   (text "MODE HIGH = standalone" (at 116.84 133.35 0)
@@
       (effects (font (size 1.27 1.27)) (justify right))
     )
-    (property "Value" "100k" (at 48.26 106.68 0)
+    (property "Value" "1k" (at 48.26 106.68 0)
       (effects (font (size 1.27 1.27)) (justify right))
     )
@@
       (effects (font (size 1.27 1.27)))
     )
-    (property "Value" "220" (at 233.68 68.58 90)
+    (property "Value" "0.22" (at 233.68 68.58 90)
       (effects (font (size 1.27 1.27)))
     )
@@
       (effects (font (size 1.27 1.27)) (justify left))
     )
-    (property "Value" "220" (at 172.72 93.98 0)
+    (property "Value" "1k" (at 172.72 93.98 0)
       (effects (font (size 1.27 1.27)) (justify left))
     )
@@
       (effects (font (size 1.27 1.27)))
     )
-    (property "Value" "100k" (at 41.91 127 90)
+    (property "Value" "1k" (at 41.91 127 90)
       (effects (font (size 1.27 1.27)))
     )
@@
       (effects (font (size 1.27 1.27)))
     )
-    (property "Value" "220" (at 233.68 54.61 90)
-      (effects (font (size 1.27 1.27)))
-    )
+    (property "Value" "0.22" (at 233.68 54.61 90)
+      (effects (font (size 1.27 1.27)))
+    )
