File: CAD/tmc_2300_standalone_bob/tmc_2300_standalone_bob.kicad_sch (KiCad schematic)
At the start: 33 parts, among them IC1 TMC2300, J1 Conn_01x04_Pin, J2 Conn_01x08_Pin, J3 Conn_01x08_Pin, J4 53261-0471

Commit message: created xiao compatible board
Parts:
- IC1: footprint footprints:QFN20_3x3_TRI -> Package_DFN_QFN:QFN-20-1EP_3x3mm_P0.45mm_EP1.6x1.6mm_ThermalVias
Changed lines of the file:
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@@
       (effects (font (size 0.9906 0.9906)))
     )
-    (property "Footprint" "footprints:QFN20_3x3_TRI" (at 207.01 66.04 0)
+    (property "Footprint" "Package_DFN_QFN:QFN-20-1EP_3x3mm_P0.45mm_EP1.6x1.6mm_ThermalVias" (at 207.01 66.04 0)
       (effects (font (size 1.27 1.27)) hide)
     )
